File: stylophone.kicad_pcb (KiCad board)
At the start: 2 copper layers, 114.3 x 86.4 mm, 25 parts, among them J1 AudioJack4, SW1 SW_MEC_5G, U1 NE555P

Commit message: stuff
Parts:
- removed D1: 1.5KExxA, Diode_THT:D_DO-201AE_P3.81mm_Vertical_AnodeUp
Routing:
- net Net-(BT1--): track 207.9 -> 10.5 mm
- net Net-(U1-R): track 196.8 -> 0.50 mm
- net Net-(U1-DIS): track 175.4 -> 0.00 mm
- net Net-(D1-A2): track 129.1 -> 4.00 mm
- net Net-(BT1-+): track 60.8 -> 0.98 mm
- net Net-(BZ1--): track 39.1 -> 0.00 mm
- net (no net): vias 1 -> 0
- added copper zone on B.Cu, net (none)
- added copper zone on F.Cu, net (none)

Commit message: yep
Parts:
- removed RV1, RV10, RV11, RV12, RV13, RV14, RV15, RV16, RV18, RV3, RV4, RV5, RV6, RV7, RV8, RV9: R_Potentiometer, Potentiometer_THT:Potentiometer_Piher_PT-6-V_Vertical
- added D1: D, Diode_THT:D_DO-201AE_P3.81mm_Vertical_AnodeUp, F.Cu at (104.1, 48.3)
- added RV_A#1: R_Potentiometer, Potentiometer_THT:Potentiometer_Piher_PT-6-V_Vertical, F.Cu at (100.4, 69.3)
- added RV_A1: R_Potentiometer, Potentiometer_THT:Potentiometer_Piher_PT-6-V_Vertical, F.Cu at (94.0, 79.5)
- added RV_B1: R_Potentiometer, Potentiometer_THT:Potentiometer_Piher_PT-6-V_Vertical, F.Cu at (106.5, 79.5)
- added RV_C#1: R_Potentiometer, Potentiometer_THT:Potentiometer_Piher_PT-6-V_Vertical, F.Cu at (37.9, 69.3)
- added RV_C1: R_Potentiometer, Potentiometer_THT:Potentiometer_Piher_PT-6-V_Vertical, F.Cu at (31.8, 79.5)
- added RV_D#1: R_Potentiometer, Potentiometer_THT:Potentiometer_Piher_PT-6-V_Vertical, F.Cu at (50.6, 69.3)
- added RV_D1: R_Potentiometer, Potentiometer_THT:Potentiometer_Piher_PT-6-V_Vertical, F.Cu at (44.2, 79.5)
- added RV_E1: R_Potentiometer, Potentiometer_THT:Potentiometer_Piher_PT-6-V_Vertical, F.Cu at (56.7, 79.5)
- added RV_F#1: R_Potentiometer, Potentiometer_THT:Potentiometer_Piher_PT-6-V_Vertical, F.Cu at (75.5, 69.3)
- added RV_F1: R_Potentiometer, Potentiometer_THT:Potentiometer_Piher_PT-6-V_Vertical, F.Cu at (69.1, 79.5)
- added RV_G#1: R_Potentiometer, Potentiometer_THT:Potentiometer_Piher_PT-6-V_Vertical, F.Cu at (87.9, 69.3)
- added RV_G1: R_Potentiometer, Potentiometer_THT:Potentiometer_Piher_PT-6-V_Vertical, F.Cu at (81.6, 79.5)
- moved BT1 6.42 mm to (41.5, 40.6)
- moved RV_C2 0.93 mm to (118.9, 79.5)
- renumbered RV17 to RV_C2
Connections:
- net Net-(BT1-+) renamed /VCC
- net Net-(D1-A2) renamed /Q
- net Net-(U1-DIS) renamed /DIS
- BT1 pad 2: Net-(BT1--) -> /GND
- BZ1 pad 2: Net-(BT1--) -> /GND
- C1 pad 1: Net-(BT1--) -> /GND
- C1 pad 2: Net-(BT1--) -> Net-(U1-THR)
- J1 pad R2: Net-(BT1--) -> /GND
- RV2 pad 1: Net-(BT1--) -> /GND
- RV_C2 pad 1: Net-(BT1--) -> /C2
- RV_C2 pad 3: Net-(U1-R) -> /GND
- SW1 pad 3: Net-(U1-R) -> /VCC_Sw
- U1 pad 1: Net-(BT1--) -> /GND
- U1 pad 2: Net-(BT1--) -> Net-(U1-THR)
- U1 pad 4: Net-(U1-R) -> /VCC_Sw
- U1 pad 6: Net-(BT1--) -> Net-(U1-THR)
- U1 pad 8: Net-(U1-R) -> /VCC_Sw
Routing:
- net /GND: track 0.00 -> 339.8 mm, vias 0 -> 2
- net /DIS: track 0.00 -> 191.5 mm, vias 0 -> 2
- net /Q: track 4.00 -> 89.0 mm, vias 0 -> 1
- net /VCC_Sw: track 0.00 -> 67.8 mm, vias 0 -> 2
- net Net-(BZ1--): track 0.00 -> 61.2 mm, vias 0 -> 1
- net /VCC: track 0.98 -> 55.8 mm
- net Net-(U1-THR): track 0.00 -> 23.9 mm
- net /D#: track 0.00 -> 19.0 mm
- net /F#: track 0.00 -> 18.9 mm
- net /G#: track 0.00 -> 18.3 mm
- net /A#: track 0.00 -> 18.3 mm
- net /C#: track 0.00 -> 18.2 mm
- net /G: track 0.00 -> 14.5 mm, vias 0 -> 1
- net /D: track 0.00 -> 14.5 mm, vias 0 -> 1
- net /A: track 0.00 -> 14.5 mm, vias 0 -> 1
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- added copper zone on F.Cu, net /A
- added copper zone on F.Cu, net /A#
- added copper zone on F.Cu, net /B
- added copper zone on F.Cu, net /C
- added copper zone on F.Cu, net /C#
- added copper zone on F.Cu, net /C2
- added copper zone on F.Cu, net /D
- added copper zone on F.Cu, net /D#
- added copper zone on F.Cu, net /E
- added copper zone on F.Cu, net /F
- added copper zone on F.Cu, net /F#
- added copper zone on F.Cu, net /G
- added copper zone on F.Cu, net /G#
- added copper zone on B.Cu, net /VCC_Sw
- added copper zone on F.Cu, net /VCC_Sw

Commit message: Add files via upload
Parts:
- BT1: footprint Battery:BatteryHolder_Keystone_1058_1x2032 -> Battery:BatteryHolder_ComfortableElectronic_CH273-2450_1x2450
- moved BT1 6.81 mm to (48.3, 40.6)
Routing:
- net /GND: track 339.8 -> 332.7 mm
- net /VCC: track 55.8 -> 62.7 mm
- net /Q: track 89.0 -> 92.4 mm
- net /F#: track 18.9 -> 18.0 mm
- removed copper zone on B.Cu, net (none)
- removed copper zone on F.Cu, net (none)
