File: stylophone.kicad_sch (KiCad schematic)
At the start: 25 parts, among them J1 AudioJack4, SW1 SW_MEC_5G, U1 NE555P

Commit message: yep
Parts:
- removed RV14, RV3, RV6, RV7: R_Potentiometer, Potentiometer_THT:Potentiometer_Piher_PT-6-V_Vertical, symbol Device:R_Potentiometer
- D1: value 1.5KExxA -> D; symbol Diode:1.5KExxA -> Device:D
- renumbered RV8 to RV_A#1, RV17 to RV_A1, RV16 to RV_B1, RV5 to RV_C#1, RV18 to RV_C1, RV15 to RV_C2, RV4 to RV_D#1, RV13 to RV_D1, RV12 to RV_E1, RV1 to RV_F#1, RV11 to RV_F1, RV9 to RV_G#1, RV10 to RV_G1
Connections:
- net DIS: now reaches RV_A#1.2, RV_A1.2, RV_B1.2, RV_C#1.2, RV_C1.2, RV_C2.2, RV_D#1.2, RV_D1.2, RV_E1.2, RV_F#1.2, RV_F1.2, RV_G#1.2, RV_G1.2, U1.7 (DIS)
- net GND: now reaches RV_A#1.3, RV_A1.3, RV_B1.3, RV_C#1.3, RV_C1.3, RV_C2.3, RV_D#1.3, RV_D1.3, RV_E1.3, RV_F#1.3, RV_F1.3, RV_G#1.3, RV_G1.3
- net GND: now also BT1.2 (-), BZ1.2 (+), C1.1, J1.R2, RV2.1, U1.1 (GND); no longer SW1.3 (B), SW1.4 (B), U1.4 (R), U1.8 (VCC)
- net Q: now reaches D1.2 (A), J1.R1, J1.T, RV2.2, U1.3 (Q)
- net VCC: now reaches BT1.1 (+), SW1.1 (A), SW1.2 (A)
- new net: C1.2, U1.2 (TR), U1.6 (THR)
- new net A: RV_A1.1
- new net A#: RV_A#1.1
- new net B: RV_B1.1
- new net C: RV_C1.1
- new net C#: RV_C#1.1
- new net C2: RV_C2.1
- new net D: RV_D1.1
- new net D#: RV_D#1.1
- new net E: RV_E1.1
- new net F: RV_F1.1
- new net F#: RV_F#1.1
- new net G: RV_G1.1
- new net G#: RV_G#1.1
- new net VCC_Sw: SW1.3 (B), SW1.4 (B), U1.4 (R), U1.8 (VCC)

Commit message: Add files via upload
Parts:
- BT1: footprint Battery:BatteryHolder_Keystone_1058_1x2032 -> Battery:BatteryHolder_ComfortableElectronic_CH273-2450_1x2450
Changed lines of the file:
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@@
       (effects (font (size 1.27 1.27)) (justify left))
     )
-    (property "Footprint" "Battery:BatteryHolder_Keystone_1058_1x2032" (at 25.4 126.746 90)
+    (property "Footprint" "Battery:BatteryHolder_ComfortableElectronic_CH273-2450_1x2450" (at 25.4 126.746 90)
       (effects (font (size 1.27 1.27)) hide)
     )
